File: discharger.sch (EAGLE design)
At the start: 72 parts, among them U1 BW6101, U10 BW6101, U11 BW6101, U12 BW6101, U2 BW6101, U3 BW6101, U4 BW6101, U5 BW6101, U6 BW6101, U7 BW6101, U8 BW6101, U9 BW6101

Commit message: use the design block
Parts:
- added JP1: LTOBMS, pinhead:PINHD-1X13
- LED1, LED10, LED11, LED12, LED2, LED3, LED4, LED5, LED6, LED7, LED8, LED9: value (none) -> ALARM
- R1, R10, R13, R16, R19, R22, R25, R28, R31, R34, R4, R7: value 47R -> 100R; device resistor:R-US_R1206W -> resistor:R-US_R0805W
- R11, R14, R17, R2, R20, R23, R26, R29, R32, R35, R5, R8: value 1K -> 47R
- R12, R15, R18, R21, R24, R27, R3, R30, R33, R36, R6, R9: value 100R -> 1K; device resistor:R-US_R1206W -> resistor:R-US_R0805W
- SJ1, SJ10, SJ11, SJ12, SJ2, SJ3, SJ4, SJ5, SJ6, SJ7, SJ8, SJ9: value (none) -> Vselect
Connections:
- removed net N$1: R3.1, U1.LED
- removed net N$2: R1.1, U1.IOUT
- removed net N$3: LED1.A, R3.2
- removed net N$5: R4.1, U2.IOUT
- removed net N$51: R31.1, U11.IOUT
- removed net N$53: R32.2, SJ11.3
- removed net N$54: R33.1, U11.LED
- removed net N$55: LED11.A, R33.2
- removed net N$7 (its old number): R2.2, SJ1.3
- new net N$6: R2.1, U1.IOUT
- new net N$66: R32.1, U11.IOUT
- new net N$68: R33.2, SJ11.3
- new net N$69: R31.1, U11.LED
- new net N$70: LED11.A, R31.2
- new net N$76: R35.1, U12.IOUT
- new net N$78: R36.2, SJ12.3
- new net N$79: R34.1, U12.LED
- new net N$80: LED12.A, R34.2
- net B-: now also JP1.7, R2.2; no longer R1.2
- net B1: now also JP1.8, R3.1, R5.2; no longer R2.1, R4.2
- net B10: now also JP1.2, R30.1, R32.2; no longer R29.1, R31.2
- net B11: now also JP1.13, R33.1, R35.2; no longer R32.1, R34.2
- net B12: now also JP1.1, R36.1; no longer R35.1
- net B2: now also JP1.6, R6.1, R8.2; no longer R5.1, R7.2
- net B3: now also JP1.9, R11.2, R9.1; no longer R10.2, R8.1
- net B4: now also JP1.5, R12.1, R14.2; no longer R11.1, R13.2
- net B5: now also JP1.10, R15.1, R17.2; no longer R14.1, R16.2
- net B6: now also JP1.4, R18.1, R20.2; no longer R17.1, R19.2
- net B7: now also JP1.11, R21.1, R23.2; no longer R20.1, R22.2
- net B8: now also JP1.3, R24.1, R26.2; no longer R23.1, R25.2
- net B9: now also JP1.12, R27.1, R29.2; no longer R26.1, R28.2
- net N$10: now also LED1.A, R1.2; no longer LED2.A, R6.2
- net N$11: now also R8.1; no longer R7.1
- net N$13: now also R9.2; no longer R8.2
- net N$14: now also R7.1; no longer R9.1
- net N$15: now also R7.2; no longer R9.2
- net N$16: now also R5.1, U2.IOUT; no longer R10.1, U4.IOUT
- net N$18: now also R6.2, SJ2.3; no longer R11.2, SJ4.3
- net N$19: now also R4.1, U2.LED; no longer R12.1, U4.LED
- net N$20: now also LED2.A, R4.2; no longer LED4.A, R12.2
- net N$21: now also R17.1, U6.IOUT; no longer R13.1, U5.IOUT
- net N$23: now also R18.2, SJ6.3; no longer R14.2, SJ5.3
- net N$24: now also R16.1, U6.LED; no longer R15.1, U5.LED
- net N$25: now also LED6.A, R16.2; no longer LED5.A, R15.2
- net N$26: now also R11.1, U4.IOUT; no longer R16.1, U6.IOUT
- net N$28: now also R12.2, SJ4.3; no longer R17.2, SJ6.3
- net N$29: now also R10.1, U4.LED; no longer R18.1, U6.LED
- net N$30: now also LED4.A, R10.2; no longer LED6.A, R18.2
- net N$31: now also R20.1; no longer R19.1
- net N$33: now also R21.2; no longer R20.2
- net N$34: now also R19.1; no longer R21.1
- net N$35: now also R19.2; no longer R21.2
- net N$36: now also R14.1, U5.IOUT; no longer R22.1, U8.IOUT
- net N$38: now also R15.2, SJ5.3; no longer R23.2, SJ8.3
- net N$39: now also R13.1, U5.LED; no longer R24.1, U8.LED
- net N$40: now also LED5.A, R13.2; no longer LED8.A, R24.2
- net N$41: now also R26.1; no longer R25.1
- net N$43: now also R27.2; no longer R26.2
- net N$44: now also R25.1; no longer R27.1
- net N$45: now also R25.2; no longer R27.2
- net N$46: now also R23.1, U8.IOUT; no longer R28.1, U10.IOUT
- net N$48: now also R24.2, SJ8.3; no longer R29.2, SJ10.3
- net N$49: now also R22.1, U8.LED; no longer R30.1, U10.LED
- net N$50: now also LED8.A, R22.2; no longer LED10.A, R30.2
- net N$56: now also R29.1, U10.IOUT; no longer R34.1, U12.IOUT
- net N$58: now also R30.2, SJ10.3; no longer R35.2, SJ12.3
- net N$59: now also R28.1, U10.LED; no longer R36.1, U12.LED
- net N$60: now also LED10.A, R28.2; no longer LED12.A, R36.2
- net N$8: now also R3.2, SJ1.3; no longer R5.2, SJ2.3
- net N$9: now also R1.1, U1.LED; no longer R6.1, U2.LED
Other:
- moved on the sheet: LED1, LED10, LED11, LED12, LED2, LED3, LED4, LED5, LED6, LED7, LED8, LED9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
